File: Rev1/BOARD1A.sch (EAGLE design)
At the start: 25 parts, among them K1 G5LE-1-VD DC12, U1 MCP23008

Commit message: Updated Design Rev2 Current
Current Design is now Rev 2. At this time looks like i can get all the
parts needed to do this one.
Parts:
- removed JMP1, JMP2, JMP3: 0R-JUMPA, jump-0r-smd:0R-JUMPA
- added ADDR1, ADDR2, ADDR3: (no value), jumper:JP2E
- added R1, R13, R14, R15, R16, R17, R18, R19, R2, R20, R21, R22, R23, R24, R25, R26, R27, R28, R29, R3, R30, R31, R32, R4, R5, R6, R7, R8: (no value), resistor:R-US_0207/12
- added R33, R34, R35, R36: (no value), SparkFun:RESISTOR1206
Connections:
- removed net N$16 (its old number): T3.B
- removed net N$18 (its old number): T4.B
- removed net N$20 (its old number): T5.B
- new net N$10: R7.1, R8.2
- new net N$2: R1.1, R2.2, R33.1, R34.2
- new net N$27: R14.1, R15.2
- new net N$28: R15.1, R16.2
- new net N$29: K4KS.P$NC, K5KS.P$COM, R16.1
- new net N$3: R2.1, R3.2, R34.1, R35.2
- new net N$30: K5KS.P$NO, R17.2
- new net N$31: R17.1, R18.2
- new net N$32: R18.1, R19.2
- new net N$33: R19.1, R20.2
- new net N$34: K5KS.P$NC, K6KS.P$COM, R20.1
- new net N$35: K6KS.P$NO, R21.2
- new net N$36: R21.1, R22.2
- new net N$37: R22.1, R23.2
- new net N$38: R23.1, R24.2
- new net N$39: K6KS.P$NC, K7KS.P$COM, R24.1
- new net N$4: R3.1, R35.1, R36.2, R4.2
- new net N$40: K7KS.P$NO, R25.2
- new net N$41: R25.1, R26.2
- new net N$42: R26.1, R27.2
- new net N$43: R27.1, R28.2
- new net N$44: K7KS.P$NC, K8KS.P$COM, R28.1
- new net N$45: K8KS.P$NO, R29.2
- new net N$46: R29.1, R30.2
- new net N$47: R30.1, R31.2
- new net N$48: R31.1, R32.2
- new net N$7: K2KS.P$NO, R5.2
- new net N$8: R6.1, R7.2
- new net N$9: R5.1, R6.2
- net +5V: now also ADDR1.3, ADDR2.3, ADDR3.3, K1KC.COILA, K2KC.COILA, K3KC.COILA, K4KC.COILA, K5KC.COILA, K6KC.COILA, K7KC.COILA, K8KC.COILA, SV1.6; no longer JMP1-0R.1, JMP2-0R.1, JMP3-0R.1, SV1.4, T1.C, T2.C, T3.C, T4.C, T5.C, T6.C, T7.C, T8.C
- net A0ADDR: now also ADDR1.2; no longer JMP1-0R.2
- net A1ADDR: now also ADDR2.2; no longer JMP2-0R.2
- net A2ADDR: now also ADDR3.2; no longer JMP3-0R.2
- net GND: now also ADDR1.1, ADDR2.1, ADDR3.1, T1.E, T2.E, T3.E, T4.E, T5.E, T6.E, T7.E, T8.E; no longer JMP1-0R.3, JMP2-0R.3, JMP3-0R.3, K1KC.COILB, K2KC.COILB, K3KC.COILB, K4KC.COILB, K5KC.COILB, K6KC.COILB, K7KC.COILB, K8KC.COILB
- net INPUT: now also SV1.4; no longer SV1.6
- net K1: now also T1.B, U1.GP3; no longer U1.GP0
- net K2: now also T2.B, U1.GP2; no longer U1.GP1
- net K3: now also T3.B, U1.GP1; no longer U1.GP2
- net K4: now also T4.B, U1.GP0; no longer U1.GP3
- net K5: now also T5.B, U1.GP4; no longer U1.GP7
- net K6: now also T6.B, U1.GP5; no longer U1.GP6
- net K7: now also T7.B, U1.GP6; no longer U1.GP5
- net K8: now also T8.B, U1.GP7; no longer U1.GP4
- net N$1: now also R1.2, R33.2; no longer R9.2
- net N$11: now also K3KC.COILB, T3.C; no longer K1KC.COILA, T1.E
- net N$12: now also K2KS.P$NC, K3KS.P$COM, R8.1; no longer T1.B
- net N$13: now also K1KC.COILB, T1.C; no longer K2KC.COILA, T2.E
- net N$14: now also K3KS.P$NO, R9.2; no longer T2.B
- net N$15: now also K2KC.COILB, T2.C; no longer K3KC.COILA, T3.E
- net N$17: now also K4KC.COILB, T4.C; no longer K4KC.COILA, T4.E
- net N$19: now also K5KC.COILB, T5.C; no longer K5KC.COILA, T5.E
- net N$21: now also K6KC.COILB, T6.C; no longer K6KC.COILA, T6.E
- net N$22: now also K3KS.P$NC, K4KS.P$COM, R12.1; no longer T6.B
- net N$23: now also K8KC.COILB, T8.C; no longer K7KC.COILA, T7.E
- net N$24: now also K4KS.P$NO, R13.2; no longer T7.B
- net N$25: now also K7KC.COILB, T7.C; no longer K8KC.COILA, T8.E
- net N$26: now also R13.1, R14.2; no longer T8.B
- net N$6: now also K2KS.P$COM, R36.1, R4.1; no longer R12.1
- net OUTPUT: now also K8KS.P$NC, R32.1
Other:
- note added: "-K1"
- note added: "-K2"
- note added: "-K3"
- note added: "-K4"
- note added: "-K5"
- note added: "-K6"
- note added: "-K7"
- note added: "-K8"
- note removed: "-R11"
- note removed: "-R12"
- note removed: "-R13"
- note removed: "-R14"
- note removed: "-R15"
- note removed: "-R16"
- note removed: "-R17"
- note removed: "-R18"
- moved on the sheet: K1KC, K1KS, K2KC, K3KC, K4KC, K5KC, K6KC, K7KC, K8KC, R10, R11, R12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
