File: Input Board/Input Board.sch (EAGLE design)
At the start: 30 parts, among them U1 MCP23008

Commit message: more work
Parts:
- removed J1, J2: (no value), SparkFun:BANANA_CONN
- removed SV1, SV2, SV3, SV4, SV5: (no value), con-lstb:MA04-2
- removed SV6: (no value), con-lstb:MA09-2
- removed SV7, SV8: (no value), con-lstb:MA05-2
Connections:
- removed net BOARDA: SV1.2, SV6.9
- removed net BOARDB: SV2.2, SV6.11
- removed net BOARDC: SV3.2, SV6.13
- removed net BOARDD: SV4.2, SV6.15
- removed net BOARDE: SV5.2, SV6.17
- removed net BOARDX1A0: SV6.8, SV7.1
- removed net BOARDX1A1: SV6.6, SV7.2
- removed net BOARDX1A2: SV6.4, SV7.4
- removed net BOARDX2A0: SV6.7, SV8.1
- removed net BOARDX2A1: SV6.5, SV8.2
- removed net BOARDX2A2: SV6.3, SV8.4
- removed net INPUT: J1.1, SV1.6
- removed net N$10: SV6.14
- removed net N$11: SV6.12
- removed net N$12: SV6.10
- removed net N$14: U1.VSS
- removed net OUTPUT: J2.1, SV8.7
- removed net OUTPUT1: SV2.5, SV3.6
- removed net OUTPUT2: SV3.5, SV4.6
- removed net OUTPUT3: SV4.5, SV5.6
- removed net OUTPUT4: SV5.5, SV7.8
- removed net OUTPUT5: SV7.7, SV8.8
- removed net OUTPUTSUB: SV1.5, SV2.6
- net +5V: now also U1.VDD; no longer SV1.4, SV2.4, SV3.4, SV4.4, SV5.4, SV6.2, SV7.6, SV8.6
- net GND: now also U1.VSS; no longer SV1.1, SV1.3, SV2.1, SV2.3, SV3.1, SV3.3, SV4.1, SV4.3, SV5.1, SV5.3, SV6.1, SV7.3, SV7.5, SV8.3, SV8.5
- net SCL: no longer SV1.7, SV2.7, SV3.7, SV4.7, SV5.7, SV6.18, SV7.9, SV8.9
- net SDA: no longer SV1.8, SV2.8, SV3.8, SV4.8, SV5.8, SV6.16, SV7.10, SV8.10
Other:
- note added: "Input Pad"
- note removed: "Bus Board"
- note removed: "MCU Connector"
- moved on the sheet: R1, R2, R3, S1, S10, S11, S12, S13, S14, S15, S16, S2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
