File: rev2/Board1a.brd (EAGLE design)
At the start: 100 x 80 mm, 57 parts, among them K1 G5LE-1-VD DC12, K5 G5LE-1-VD DC12, U1 MCP23008

Commit message: more work
Changed lines of the file:
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@@
 <attribute name="MF" value="" x="15.875" y="66.675" size="1.778" layer="27" display="off"/>
 <attribute name="OC_FARNELL" value="unknown" x="15.875" y="66.675" size="1.778" layer="27" display="off"/>
-<attribute name="NAME" x="10.414" y="64.135" size="0.8128" layer="25" ratio="10" rot="R90"/>
+<attribute name="NAME" x="10.414" y="66.675" size="0.8128" layer="25" ratio="10" rot="R90"/>
 <attribute name="VALUE" x="15.875" y="62.484" size="1.27" layer="27" ratio="10"/>
 </element>
@@
 </element>
 <element name="ADDR1" library="jumper" package="JP2" value="" x="12.7" y="54.61" smashed="yes" rot="R180">
-<attribute name="NAME" x="16.891" y="54.356" size="0.8128" layer="25" ratio="10" rot="R270"/>
+<attribute name="NAME" x="16.891" y="56.261" size="0.8128" layer="25" ratio="10" rot="R270"/>
 <attribute name="VALUE" x="16.256" y="58.928" size="1.27" layer="27" ratio="10" rot="R180"/>
 </element>
 <element name="ADDR2" library="jumper" package="JP2" value="" x="12.7" y="48.895" smashed="yes" rot="R180">
-<attribute name="NAME" x="16.891" y="49.276" size="0.8128" layer="25" ratio="10" rot="R270"/>
+<attribute name="NAME" x="16.891" y="50.546" size="0.8128" layer="25" ratio="10" rot="R270"/>
 <attribute name="VALUE" x="16.256" y="53.213" size="1.27" layer="27" ratio="10" rot="R180"/>
 </element>
@@
 <contactref element="U1" pad="P$1"/>
 <wire x1="17.145" y1="65.405" x2="17.145" y2="45.72" width="0.254" layer="16"/>
-<wire x1="17.145" y1="45.72" x2="17.78" y2="45.085" width="0.254" layer="16"/>
-<wire x1="17.78" y1="45.085" x2="19.05" y2="45.085" width="0.254" layer="16"/>
+<wire x1="17.145" y1="45.72" x2="19.05" y2="45.085" width="0.254" layer="16"/>
 </signal>
 <signal name="SDA">
