File: rev2/Board1a.sch (EAGLE design)
At the start: 57 parts, among them K1 G5LE-1-VD DC12, K5 G5LE-1-VD DC12, U1 MCP23008

Commit message: more work
Other:
- note added: "EXP X1"
- note added: "EXP X2"
- note added: "Input Board (Hardwire)"
Changed lines of the file:
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@@
 <wire x1="127" y1="63.5" x2="127" y2="60.96" width="0.1524" layer="97"/>
 <wire x1="127" y1="60.96" x2="132.08" y2="60.96" width="0.1524" layer="97"/>
-<wire x1="132.08" y1="60.96" x2="137.16" y2="60.96" width="0.1524" layer="97"/>
 <wire x1="137.16" y1="60.96" x2="142.24" y2="60.96" width="0.1524" layer="97"/>
 <text x="129.54" y="67.31" size="1.778" layer="97" align="center">0</text>
@@
 <wire x1="147.32" y1="73.66" x2="152.4" y2="73.66" width="0.1524" layer="97"/>
 <wire x1="152.4" y1="73.66" x2="157.48" y2="73.66" width="0.1524" layer="97"/>
-<wire x1="182.88" y1="60.96" x2="157.48" y2="60.96" width="0.1524" layer="97"/>
+<wire x1="182.88" y1="60.96" x2="177.8" y2="60.96" width="0.1524" layer="97"/>
+<wire x1="172.72" y1="60.96" x2="167.64" y2="60.96" width="0.1524" layer="97"/>
+<wire x1="162.56" y1="60.96" x2="157.48" y2="60.96" width="0.1524" layer="97"/>
 <wire x1="152.4" y1="60.96" x2="147.32" y2="60.96" width="0.1524" layer="97"/>
 <wire x1="147.32" y1="60.96" x2="147.32" y2="63.5" width="0.1524" layer="97"/>
@@
 <wire x1="157.48" y1="73.66" x2="162.56" y2="73.66" width="0.1524" layer="97"/>
 <wire x1="162.56" y1="73.66" x2="167.64" y2="73.66" width="0.1524" layer="97"/>
-<wire x1="167.64" y1="73.66" x2="172.72" y2="73.66" width="0.1524" layer="97"/>
 <wire x1="172.72" y1="73.66" x2="177.8" y2="73.66" width="0.1524" layer="97"/>
 <wire x1="177.8" y1="73.66" x2="182.88" y2="73.66" width="0.1524" layer="97"/>
 <wire x1="182.88" y1="73.66" x2="182.88" y2="71.12" width="0.1524" layer="97"/>
-<text x="129.54" y="59.69" size="1.778" layer="97" align="center">1</text>
-<text x="134.62" y="59.69" size="1.778" layer="97" align="center">0</text>
-<text x="139.7" y="59.69" size="1.778" layer="97" align="center">1</text>
-<text x="129.54" y="57.15" size="1.778" layer="97" align="center">1</text>
-<text x="134.62" y="57.15" size="1.778" layer="97" align="center">1</text>
-<text x="139.7" y="57.15" size="1.778" layer="97" align="center">0</text>
 <text x="165.1" y="67.31" size="0.6096" layer="97" ratio="10" align="center">1K</text>
-<text x="129.54" y="54.61" size="1.778" layer="97" align="center">1</text>
-<text x="134.62" y="54.61" size="1.778" layer="97" align="center">1</text>
-<text x="139.7" y="54.61" size="1.778" layer="97" align="center">1</text>
 <text x="144.78" y="64.77" size="0.6096" layer="97" ratio="10" align="center">10K</text>
 <text x="165.1" y="64.77" size="0.6096" layer="97" ratio="10" align="center">100K</text>
@@
 <wire x1="182.88" y1="68.58" x2="182.88" y2="66.04" width="0.1524" layer="97"/>
 <wire x1="182.88" y1="66.04" x2="182.88" y2="63.5" width="0.1524" layer="97"/>
-<wire x1="182.88" y1="63.5" x2="182.88" y2="60.96" width="0.1524" layer="97"/>
-<wire x1="127" y1="60.96" x2="127" y2="58.42" width="0.1524" layer="97"/>
-<wire x1="127" y1="58.42" x2="127" y2="55.88" width="0.1524" layer="97"/>
-<wire x1="127" y1="55.88" x2="127" y2="53.34" width="0.1524" layer="97"/>
-<wire x1="127" y1="53.34" x2="132.08" y2="53.34" width="0.1524" layer="97"/>
-<wire x1="132.08" y1="53.34" x2="137.16" y2="53.34" width="0.1524" layer="97"/>
-<wire x1="137.16" y1="53.34" x2="142.24" y2="53.34" width="0.1524" layer="97"/>
-<wire x1="142.24" y1="53.34" x2="147.32" y2="53.34" width="0.1524" layer="97"/>
-<wire x1="147.32" y1="53.34" x2="152.4" y2="53.34" width="0.1524" layer="97"/>
-<wire x1="152.4" y1="53.34" x2="157.48" y2="53.34" width="0.1524" layer="97"/>
-<wire x1="157.48" y1="53.34" x2="162.56" y2="53.34" width="0.1524" layer="97"/>
-<wire x1="162.56" y1="53.34" x2="167.64" y2="53.34" width="0.1524" layer="97"/>
-<wire x1="167.64" y1="53.34" x2="172.72" y2="53.34" width="0.1524" layer="97"/>
-<wire x1="172.72" y1="53.34" x2="177.8" y2="53.34" width="0.1524" layer="97"/>
-<wire x1="177.8" y1="53.34" x2="182.88" y2="53.34" width="0.1524" layer="97"/>
-<wire x1="127" y1="58.42" x2="182.88" y2="58.42" width="0.1524" layer="97"/>
-<wire x1="182.88" y1="58.42" x2="182.88" y2="60.96" width="0.1524" layer="97"/>
-<wire x1="127" y1="55.88" x2="182.88" y2="55.88" width="0.1524" layer="97"/>
-<wire x1="182.88" y1="55.88" x2="182.88" y2="58.42" width="0.1524" layer="97"/>
-<wire x1="182.88" y1="55.88" x2="182.88" y2="53.34" width="0.1524" layer="97"/>
-<wire x1="157.48" y1="60.96" x2="157.48" y2="53.34" width="0.1524" layer="97"/>
-<wire x1="152.4" y1="60.96" x2="152.4" y2="53.34" width="0.1524" layer="97"/>
-<wire x1="147.32" y1="60.96" x2="147.32" y2="53.34" width="0.1524" layer="97"/>
-<wire x1="142.24" y1="60.96" x2="142.24" y2="53.34" width="0.1524" layer="97"/>
-<wire x1="137.16" y1="60.96" x2="137.16" y2="53.34" width="0.1524" layer="97"/>
-<wire x1="132.08" y1="60.96" x2="132.08" y2="53.34" width="0.1524" layer="97"/>
 <wire x1="147.32" y1="63.5" x2="182.88" y2="63.5" width="0.1524" layer="97"/>
 <wire x1="147.32" y1="66.04" x2="182.88" y2="66.04" width="0.1524" layer="97"/>
@@
 <text x="160.02" y="73.66" size="1.778" layer="97" rot="R90">-K4</text>
 <text x="180.34" y="73.66" size="1.778" layer="97" rot="R90">-K8</text>
-<wire x1="162.56" y1="73.66" x2="162.56" y2="53.34" width="0.1524" layer="97"/>
-<wire x1="167.64" y1="73.66" x2="167.64" y2="53.34" width="0.1524" layer="97"/>
-<wire x1="172.72" y1="73.66" x2="172.72" y2="53.34" width="0.1524" layer="97"/>
-<wire x1="177.8" y1="73.66" x2="177.8" y2="53.34" width="0.1524" layer="97"/>
 <wire x1="55.88" y1="35.56" x2="0" y2="35.56" width="0.1524" layer="97"/>
 <wire x1="55.88" y1="86.36" x2="124.46" y2="86.36" width="0.1524" layer="97"/>
@@
 <text x="175.26" y="62.23" size="0.6096" layer="97" ratio="10" align="center">20M</text>
 <text x="180.34" y="62.23" size="0.6096" layer="97" ratio="10" align="center">40M</text>
+<wire x1="162.56" y1="73.66" x2="162.56" y2="60.96" width="0.1524" layer="97"/>
+<wire x1="167.64" y1="60.96" x2="167.64" y2="73.66" width="0.1524" layer="97"/>
+<wire x1="167.64" y1="73.66" x2="172.72" y2="73.66" width="0.1524" layer="97"/>
+<wire x1="172.72" y1="73.66" x2="172.72" y2="60.96" width="0.1524" layer="97"/>
+<wire x1="172.72" y1="60.96" x2="177.8" y2="60.96" width="0.1524" layer="97"/>
+<wire x1="177.8" y1="60.96" x2="177.8" y2="73.66" width="0.1524" layer="97"/>
+<wire x1="182.88" y1="60.96" x2="182.88" y2="63.5" width="0.1524" layer="97"/>
+<text x="129.54" y="59.69" size="1.778" layer="97" align="center">1</text>
+<text x="139.7" y="59.69" size="1.778" layer="97" align="center">1</text>
+<text x="134.62" y="59.69" size="1.778" layer="97" align="center">0</text>
+<text x="129.54" y="57.15" size="1.778" layer="97" align="center">1</text>
+<text x="134.62" y="57.15" size="1.778" layer="97" align="center">1</text>
+<text x="139.7" y="57.15" size="1.778" layer="97" align="center">0</text>
+<text x="139.7" y="54.61" size="1.778" layer="97" align="center">1</text>
+<text x="134.62" y="54.61" size="1.778" layer="97" align="center">1</text>
+<text x="129.54" y="54.61" size="1.778" layer="97" align="center">1</text>
+<text x="142.748" y="59.69" size="1.778" layer="97" align="center-left">EXP X1</text>
+<text x="142.748" y="57.15" size="1.778" layer="97" align="center-left">EXP X2</text>
+<text x="142.748" y="54.61" size="1.778" layer="97" align="center-left">Input Board (Hardwire)</text>
+<wire x1="127" y1="60.96" x2="127" y2="58.42" width="0.1524" layer="97"/>
+<wire x1="127" y1="58.42" x2="127" y2="55.88" width="0.1524" layer="97"/>
+<wire x1="132.08" y1="53.34" x2="137.16" y2="53.34" width="0.1524" layer="97"/>
+<wire x1="142.24" y1="53.34" x2="182.88" y2="53.34" width="0.1524" layer="97"/>
+<wire x1="182.88" y1="53.34" x2="182.88" y2="55.88" width="0.1524" layer="97"/>
+<wire x1="182.88" y1="55.88" x2="182.88" y2="58.42" width="0.1524" layer="97"/>
+<wire x1="182.88" y1="58.42" x2="182.88" y2="60.96" width="0.1524" layer="97"/>
+<wire x1="167.64" y1="60.96" x2="162.56" y2="60.96" width="0.1524" layer="97"/>
+<wire x1="142.24" y1="60.96" x2="142.24" y2="58.42" width="0.1524" layer="97"/>
+<wire x1="142.24" y1="55.88" x2="142.24" y2="53.34" width="0.1524" layer="97"/>
+<wire x1="142.24" y1="53.34" x2="137.16" y2="53.34" width="0.1524" layer="97"/>
+<wire x1="137.16" y1="53.34" x2="137.16" y2="60.96" width="0.1524" layer="97"/>
+<wire x1="137.16" y1="60.96" x2="132.08" y2="60.96" width="0.1524" layer="97"/>
+<wire x1="132.08" y1="60.96" x2="132.08" y2="53.34" width="0.1524" layer="97"/>
+<wire x1="132.08" y1="53.34" x2="127" y2="53.34" width="0.1524" layer="97"/>
+<wire x1="127" y1="53.34" x2="127" y2="55.88" width="0.1524" layer="97"/>
+<wire x1="127" y1="55.88" x2="142.24" y2="55.88" width="0.1524" layer="97"/>
+<wire x1="142.24" y1="55.88" x2="142.24" y2="58.42" width="0.1524" layer="97"/>
+<wire x1="142.24" y1="58.42" x2="127" y2="58.42" width="0.1524" layer="97"/>
+<wire x1="142.24" y1="58.42" x2="182.88" y2="58.42" width="0.1524" layer="97"/>
+<wire x1="142.24" y1="55.88" x2="182.88" y2="55.88" width="0.1524" layer="97"/>
 </plain>
 <instances>
